File: kicad/main_board/main_board.kicad_sch (KiCad schematic)
At the start: 42 parts, among them J1 Barrel_Jack, J2 MSTBA 5.08mm 01x02, J3 61400826021, J4 0.1" Male 01x03, J5 0.1" Male 01x03, J6 Conn_ARM_JTAG_SWD_10, Q1 FQP27P06, U2 Pico

Commit message: First working version
Parts:
- removed J6: Conn_ARM_JTAG_SWD_10, Connector_PinHeader_1.27mm:PinHeader_2x05_P1.27mm_Vertical_SMD, symbol Connector:Conn_ARM_JTAG_SWD_10
- removed R6: 10k, Capacitor_SMD:C_0603_1608Metric, symbol Device:R_US
- removed TP1: TestPoint, TestPoint:TestPoint_Pad_2.0x2.0mm, symbol Connector:TestPoint
- added C11, C12, C13: 22uF X7R 25V, Capacitor_SMD:C_1210_3225Metric, symbol Device:C
- added GRAPHIC1: Graphic, Custom_Graphic:bird_with_pants_small_flipped, symbol Custom_Placeholder:Graphic
- added H1, H2, H3, H4: MountingHole, MountingHole:MountingHole_3.2mm_M3, symbol Mechanical:MountingHole
- added PCB1: PCB, Custom_Graphic:PCB_PN_REV, symbol Custom_Placeholder:PCB
- C10: value 47pF -> DNP
- D1: footprint Diode_SMD:D_MicroMELF -> Diode_SMD:D_MiniMELF
- D2: MPN https://fscdn.rohm.com/en/products/databook/datasheet/opto/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 -> SK34A-LTP
- R1, R4, R5: footprint Capacitor_SMD:C_0603_1608Metric -> Resistor_SMD:R_0603_1608Metric
- R2: value 15k 1% -> 110k 1%; footprint Capacitor_SMD:C_0603_1608Metric -> Resistor_SMD:R_0603_1608Metric
- R3: value 110k 1% -> 15k 1%; footprint Capacitor_SMD:C_0603_1608Metric -> Resistor_SMD:R_0603_1608Metric
- TP1, TP3: MPN (none) -> DNP
- U1: value ~ -> AOZ6605PI-1; footprint Package_SO:SOIC-8-1EP_3.9x4.9mm_P1.27mm_EP2.29x3mm_ThermalVias -> Custom_Package_SO:SOIC-8-1EP_3.9x4.9mm_P1.27mm_EP2.29x3mm_ThermalVias; MPN (none) -> AOZ6605PI-1; Standard Cost (none) -> 0.33
- U2: footprint Custom_Module:RPi_Pico_SMD_TH -> Custom_Module:RPi_Pico_TH_Socket; symbol Custom_MCU:Pico -> Custom_MCU:Pico_H; MPN SC0915 -> SC0917
Connections:
- net +5V: now also J4.3 (Pin_3), J5.3 (Pin_3), C11.1, C12.1, C13.1; no longer J4.1 (Pin_1), J5.1 (Pin_1)
- net GND: now also J4.1 (Pin_1), J5.1 (Pin_1), C11.2, C12.2, C13.2; no longer J4.3 (Pin_3), J5.3 (Pin_3), U2.42 (GND)
- net LED_LEFT_DATA: now also U2.22 (GPIO17); no longer U2.1 (GPIO0)
- net LED_RIGHT_DATA: now also U2.21 (GPIO16); no longer U2.2 (GPIO1)
- net ~{RESET}: no longer names the net of U2.30 (RUN)
- no-connect marks 32 -> 30
Other:
- company: (none) -> Pants for Birds
- title: (none) -> Drill Press Camera Main Board
- moved on the sheet: D2, D3, J2, J3, J4, J5, R7, TP1
